File: hardware/pdsupply-duo/pdsupply-duo.kicad_pcb (KiCad board)
At the start: 2 copper layers, 0 parts

Commit message: Added usb PD interface
Parts:
- added C2: .1uF, Capacitor_SMD:C_0603_1608Metric, F.Cu at (190.5, 124.5)
- added C3: .1uF, Capacitor_SMD:C_0603_1608Metric, F.Cu at (171.4, 143.6)
- added C4: 4.7uF, Capacitor_SMD:C_0603_1608Metric, F.Cu at (178.4, 136.5)
- added J1: USB4505-03-0-A_REVA, USB4505-03-0-A_REVA-usbport:GCT_USB4505-03-0-A_REVA, F.Cu at (162.5, 142.3)
- added U1: LTM8074IY, LTM8074IY_PBF-buck:BGA25C65P5X5_400X400X198N, F.Cu at (172.9, 138.8)
- added U2: BMD-340-A-R, BMD-340-A-R-nrf52:RIGADO_BMD-340-A-R, F.Cu at (163.7, 129.1)
- added U3: BMD-340-A-R, BMD-340-A-R-nrf52:RIGADO_BMD-340-A-R, F.Cu at (213.4, 99.1)
Other:
- board outline added: 12.9 x 6.6 mm
